File: v3_rp2040/board/calipers_in.kicad_sch (KiCad schematic)
At the start: 14 parts, among them IC1 LM393, J8 USB_A, U11 USBLC6-2SC6

Commit message: v3: resolve missing footprints, fix part data and datasheet links
- Add project footprint library lib/footprint.pretty with RP2040-QFN-56,
  USB-C-SMD_TYPE-C-16P-1 and OSC-SMD_4P-L3.2-W2.5-BL (from
  moba-hausbeleuchtung) and USB_A_Upright_C26235 (from v2). Upgraded to
  current format, 3D model paths made project-relative, USB-A footprint
  checked against the C26235 drawing and given a courtyard.
- U2: EL357N from the old v2 library replaced by stock LTV-817S,
  matching U15-U17.
- U4 (LM358DR2G): assign SOIC-8_3.9x4.9mm_P1.27mm, checked against
  onsemi case 751-07.
- U5: switch to W25Q128JVSIQ (C97521, JLC basic part), stock
  Memory_Flash:W25Q128JVS symbol, footprint renamed to
  SOIC-8_5.3x5.3mm_P1.27mm (checked against Winbond 208-mil package).
  Netlist unchanged.
- Replace expiring JLC OSS datasheet links (and a dead szlcsc link) with
  permanent lcsc.com/datasheet/<C#>.pdf URLs.

Co-Authored-By: Claude Opus 5.5 <noreply@anthropic.com>
Parts:
- J8: footprint Lathecontrol_STM32:USB_A_Upright_C26235 -> footprint:USB_A_Upright_C26235
