File: v3_rp2040/board/calipers_in.kicad_sch (KiCad schematic)
At the start: 14 parts, among them IC1 LM393, J8 USB_A, U11 USBLC6-2SC6

Commit message: schematic bla
Parts:
- renumbered C21 to C28, C22 to C29, C23 to C30, J8 to J9, R20 to R29, R21 to R30, R22 to R31, R23 to R32, R24 to R33, R25 to R34, R26 to R35, R27 to R36, U11 to U14
