File: v3_rp2040/board/lathecontrol_v3.kicad_sch (KiCad schematic)
At the start: 46 parts, among them J1 Conn_01x06_Male, J14 Conn_01x04_Male, J4 USB_B_Micro, J5 Conn_01x05_Male, J6 Conn_01x05_Male, J7 Conn_01x14_Female, Q2 MMBT3904, U1 STM32F103RBTx, U2 6N137, U3 LM2904, U4 LM317_TO-252, U5 AMS1117-3.3, U6 Everlight_Elec_EL357N, Y1 8MHz

Commit message: schematic work
Parts:
- removed C1, C3: 30p, Capacitor_SMD:C_0603_1608Metric, symbol Device:C
- removed C2, C4, C5, C7: 100n, Capacitor_SMD:C_0603_1608Metric, symbol Device:C
- removed D2: RED, LED_SMD:LED_0603_1608Metric, symbol Device:LED
- removed J1: Conn_01x06_Male, Connector_PinHeader_2.54mm:PinHeader_1x06_P2.54mm_Vertical, symbol Connector:Conn_01x06_Male
- removed J4: USB_B_Micro, Lathecontrol_STM32:USB_Micro-B_SHOU_HAN_MicroXNJ, symbol lathecontrol_stm32-rescue:USB_B_Micro-Connector
- removed JP1: BOOTSEL, Connector_PinHeader_2.54mm:PinHeader_1x02_P2.54mm_Horizontal, symbol Jumper:Jumper_2_Open
- removed R1: 10k, Resistor_SMD:R_0603_1608Metric, symbol Device:R
- removed R3: 1k5, Resistor_SMD:R_0603_1608Metric, symbol Device:R
- removed R4: 240, Resistor_SMD:R_0603_1608Metric, symbol Device:R
- removed U1: STM32F103RBTx, Package_QFP:LQFP-64_10x10mm_P0.5mm, symbol MCU_ST_STM32F1:STM32F103RBTx
- removed Y1: 8MHz, Crystal:Crystal_SMD_5032-2Pin_5.0x3.2mm, symbol Device:Crystal
- added C10, C11, C13, C14, C15, C16, C17, C25, C28: 100n, Capacitor_SMD:C_0402_1005Metric, symbol Device:C_Small
- added C22, C24: 1u, Capacitor_SMD:C_0402_1005Metric, symbol Device:C_Small
- added C26, C27: 22p, Capacitor_SMD:C_0402_1005Metric, symbol Device:C_Small
- added D8, D9: D, Diode_SMD:D_SOD-123F, symbol Device:D
- added J13: SWD, Connector_PinHeader_2.54mm:PinHeader_2x03_P2.54mm_Vertical, symbol Connector_Generic:Conn_02x03_Odd_Even
- added J2: I2C_EXP, Connector_PinHeader_2.54mm:PinHeader_1x04_P2.54mm_Vertical, symbol Connector:Conn_01x04_Socket
- added J8: DEBUG, Connector_PinHeader_2.54mm:PinHeader_1x04_P2.54mm_Vertical, symbol Connector:Conn_01x04_Socket
- added JP1: Auto-Bootsel, Resistor_SMD:R_0603_1608Metric, symbol Jumper:SolderJumper_2_Bridged
- added Q1: MMBT3904, Package_TO_SOT_SMD:SOT-23, symbol Transistor_BJT:MMBT3904
- added R13, R14, R15, R16, R28, R29: 5k1, Resistor_SMD:R_0603_1608Metric, symbol Device:R_Small
- added R17, R18: 22, Resistor_SMD:R_0402_1005Metric, symbol Device:R_Small
- added R19, R23: 1k, Resistor_SMD:R_0402_1005Metric, symbol Device:R_Small
- added R24, R27: 27, Resistor_SMD:R_0603_1608Metric, symbol Device:R_Small
- added R30: 10k, Resistor_SMD:R_0402_1005Metric, symbol Device:R
- added TP1, TP2: TestPoint, TestPoint:TestPoint_Pad_D1.5mm, symbol Connector:TestPoint
- added U10: RP2040, footprint:RP2040-QFN-56, symbol MCU_RaspberryPi:RP2040
- added U11: W25Q128JVS, Package_SO:SOIC-8_5.23x5.23mm_P1.27mm, symbol _JLC_Flash_16MB:W25Q16JVSSIQ
- added U7, U9: TYPEC-304-ACP16, footprint:USB-C-SMD_TYPE-C-16P-1, symbol _JLC_USB_TYPEC:TYPEC-304-ACP16
- added U8: USBLC6-2SC6, Package_TO_SOT_SMD:SOT-23-6, symbol Power_Protection:USBLC6-2SC6
- added Y1: 12 Mhz, footprint:OSC-SMD_4P-L3.2-W2.5-BL, symbol Device:Crystal_GND24
Connections:
- net +3V3: now also C13.1, C14.1, C15.1, C16.1, C17.1, C24.1, C25.1, C28.1, J13.2 (Pin_2), R28.1, R29.1, U10.1 (IOVDD), U10.10 (IOVDD), U10.22 (IOVDD), U10.33 (IOVDD), U10.42 (IOVDD), U10.43 (ADC_AVDD), U10.44 (VREG_IN), U10.48 (USB_VDD), U10.49 (IOVDD), U11.8 (VCC)
- net +5V: now also D9.2 (A), J13.4 (Pin_4), J2.1 (Pin_1), U9.A4B9 (VBUS), U9.B4A9 (VBUS); no longer C20.1, U5.3 (VI)
- net GND: now also C10.2, C11.2, C13.2, C14.2, C15.2, C16.2, C17.2, C22.2, C24.2, C25.2, C26.2, C27.2, C28.2, J13.6 (Pin_6), J2.4 (Pin_4), J8.4 (Pin_4), Q1.2 (E), R13.1, R14.2, R15.1, R16.2, U10.19 (TESTEN), U10.57 (GND), U11.4 (GND), U7.A1B12 (GND), U7.B1A12 (GND), U7.EP, U8.2 (GND), U9.A1B12 (GND), U9.B1A12 (GND), U9.EP, Y1.2, Y1.4
- net SWCLK: now also J13.5 (Pin_5), U10.24 (SWCLK)
- net SWDIO: now also J13.3 (Pin_3), U10.25 (SWD)
- new net: R24.1, U10.36 (GPIO24)
- new net: R13.2, U7.A5 (CC1)
- new net: R14.1, U7.B5 (CC2)
- new net: Q1.1 (B), R30.2
- new net: JP1.1 (A), Q1.3 (C)
- new net: C20.1, D8.1 (K), D9.1 (K), U5.3 (VI)
- new net: R27.1, U10.37 (GPIO25)
- new net: C27.1, R23.1, Y1.3
- new net: R16.1, U9.B5 (CC2)
- new net: R15.2, U9.A5 (CC1)
- new net +1V1: C10.1, C11.1, C22.1, TP1.1, U10.23 (DVDD), U10.45 (VREG_VOUT), U10.50 (DVDD)
- new net BOOTSEL: J8.3 (Pin_3), JP1.2 (B), R19.1
- new net DBG_RX: J8.1 (Pin_1), U10.3 (GPIO1)
- new net DBG_TX: J8.2 (Pin_2), U10.2 (GPIO0)
- new net I2C0_SCL: J2.3 (Pin_3), R27.2, R29.2
- new net I2C0_SDA: J2.2 (Pin_2), R24.2, R28.2
- new net LED: U10.14 (GPIO11)
- new net QSPI_SCLK: U10.52 (QSPI_SCLK), U11.6 (CLK)
- new net QSPI_SD0: U10.53 (QSPI_SD0), U11.5 (DI/IO0)
- new net QSPI_SD1: U10.55 (QSPI_SD1), U11.2 (DO/IO1)
- new net QSPI_SD2: U10.54 (QSPI_SD2), U11.3 (IO2)
- new net QSPI_SD3: U10.51 (QSPI_SD3), U11.7 (IO3)
- new net QSPI_SS: R19.2, U10.56 (QSPI_SS), U11.1 (/CS)
- new net RUN: J13.1 (Pin_1), U10.26 (RUN)
- new net USB_DN1: U7.A7 (D-), U7.B7 (D-), U8.4 (I/O2)
- new net USB_DN2: R18.2, U8.3 (I/O2)
- new net USB_DN3: R18.1, U10.46 (USB_DM)
- new net USB_DP1: U7.A6 (D+), U7.B6 (D+), U8.6 (I/O1)
- new net USB_DP2: R17.1, U8.1 (I/O1)
- new net USB_DP3: R17.2, U10.47 (USB_DP)
- new net VBUS: D8.2 (A), R30.1, TP2.1, U7.A4B9 (VBUS), U7.B4A9 (VBUS), U8.5 (VBUS)
- new net XIN: C26.1, U10.20 (XIN), Y1.1
- new net XOUT: R23.2, U10.21 (XOUT)
- no-connect marks 16 -> 30
Other:
- sheet Measurestick Input 1 renamed Calipers1
- sheet Measurestick Input 2 renamed Calipers2
- sheet Measurestick Input 3 renamed Calipers3
- sheet Measurestick Input 4 renamed Calipers4
- sheet Calipers1: file measurestick_single.kicad_sch -> calipers_in.kicad_sch
- sheet Calipers2: file measurestick_single.kicad_sch -> calipers_in.kicad_sch
- sheet Calipers3: file measurestick_single.kicad_sch -> calipers_in.kicad_sch
- sheet Calipers4: file measurestick_single.kicad_sch -> calipers_in.kicad_sch
- note added: "Auto Bootsel"
- note added: "CRY has 20pF load capacitance External load capacitance: 2*(20pF - 5pF) = 30pF"
- note added: "DEBUG / PROG"
- note added: "Flash 16 MBit (2MB)"
- note added: "I2C"
- note added: "Maybe use 128MBit (16MB) C97521 instead (Basic Part)? 49ct@30pcs vs 19ct@36pcs"
- note added: "RP2040"
- note added: "USB-C (Power / RUN)"
- note added: "USB-C (Programming)"
- note removed: "C1 = C3 = 2 * (CL - Cstray) CL = 20 pF (Cystal Datasheet) Cstray ca. 5 pF"
- note removed: "PC13, PC14, PC15 can source / sink +/-3mA only!"
- note removed: "Programming Interface (SWD)"
- note removed: "USB Input"
- note removed: "uCPU STM32f103RB, Arm Cortex-M3 MCU with 128 Kbytes of Flash memory, 72 MHz CPU"
- moved on the sheet: C12, C18, C19, C20, C21, C23, C6, D5, D6, H1, H2, H3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

Commit message: more schematic work
Parts:
- removed C6: 100n, Capacitor_SMD:C_0603_1608Metric, symbol Device:C
- removed R2: 180, Resistor_SMD:R_0603_1608Metric, symbol Device:R
- removed U2: 6N137, Package_DIP:DIP-8_W7.62mm, symbol Isolator:6N137
- removed U3: LM2904, symbol Amplifier_Operational:LM2904
- added U15, U16, U17: LTV-817S-TA1-C, Package_DIP:SMDIP-4_W9.53mm, symbol Isolator:LTV-817S
- added U3: 78L05G-AB3-R, Package_TO_SOT_SMD:SOT-89-3, symbol Regulator_Linear:L78L05_SOT89
- added U4: LM358DR2G, symbol Amplifier_Operational:LM358
- renumbered C10 to C1, C22 to C10, C24 to C11, C23 to C12, C26 to C14, C27 to C15, C28 to C16, C20 to C17, C21 to C18, C18 to C19, C11 to C2, C19 to C20, C13 to C3, C14 to C4, C15 to C5, C16 to C6, C17 to C7, C25 to C8, C12 to C9, D9 to D1, D8 to D2, D5 to D3, D6 to D4, J5 to J1, J7 to J2, J6 to J3, J14 to J4, J2 to J5, J13 to J6, J8 to J7, Q2 to Q1, Q1 to Q2, R17 to R1, R23 to R10, R19 to R11, R30 to R12, R14 to R13, R16 to R14, R13 to R15, R15 to R16, R22 to R17, R20 to R18, R21 to R19, R18 to R2, R25 to R3, R28 to R4, R29 to R5, R26 to R6, R24 to R7, R27 to R8, U10 to U1, U8 to U10, U6 to U2, U11 to U5, U7 to U6, U9 to U7, U5 to U8, U4 to U9
Connections:
- no-connect marks 30 -> 27
Other:
- note removed: "4...20mA output for frequency converter"
- note removed: "Max 7V"
