File: v3_rp2040/board/lathecontrol_v3.kicad_sch (KiCad schematic)
At the start: 73 parts, among them J1 Conn_01x05_Male, J2 Conn_01x14_Female, J3 Conn_01x05_Male, J4 Conn_01x04_Male, J5 I2C_EXP, J6 SWD, J7 DEBUG, Q1 MMBT3904, Q2 MMBT3904, U1 RP2040, U10 USBLC6-2SC6, U15 LTV-817S-TA1-C, U16 LTV-817S-TA1-C, U17 LTV-817S-TA1-C, U2 Everlight_Elec_EL357N, U3 78L05G-AB3-R, U4 LM358DR2G, U5 W25Q128JVS, U6 TYPEC-304-ACP16, U7 TYPEC-304-ACP16, U8 AMS1117-3.3, U9 LM317_TO-252, Y1 12 Mhz

Commit message: v3: resolve missing footprints, fix part data and datasheet links
- Add project footprint library lib/footprint.pretty with RP2040-QFN-56,
  USB-C-SMD_TYPE-C-16P-1 and OSC-SMD_4P-L3.2-W2.5-BL (from
  moba-hausbeleuchtung) and USB_A_Upright_C26235 (from v2). Upgraded to
  current format, 3D model paths made project-relative, USB-A footprint
  checked against the C26235 drawing and given a courtyard.
- U2: EL357N from the old v2 library replaced by stock LTV-817S,
  matching U15-U17.
- U4 (LM358DR2G): assign SOIC-8_3.9x4.9mm_P1.27mm, checked against
  onsemi case 751-07.
- U5: switch to W25Q128JVSIQ (C97521, JLC basic part), stock
  Memory_Flash:W25Q128JVS symbol, footprint renamed to
  SOIC-8_5.3x5.3mm_P1.27mm (checked against Winbond 208-mil package).
  Netlist unchanged.
- Replace expiring JLC OSS datasheet links (and a dead szlcsc link) with
  permanent lcsc.com/datasheet/<C#>.pdf URLs.

Co-Authored-By: Claude Opus 5.5 <noreply@anthropic.com>
Parts:
- U2: value Everlight_Elec_EL357N -> LTV-817S-TA1-C; footprint Lathecontrol_STM32:SOP-4_4.1x4.4x2.54P -> Package_DIP:SMDIP-4_W9.53mm; symbol Lathecontrol_STM32:Everlight_Elec_EL357N -> Isolator:LTV-817S; LCSC C6649 -> C109227
- U4: footprint (none) -> Package_SO:SOIC-8_3.9x4.9mm_P1.27mm
- U5: value W25Q128JVS -> W25Q128JVSIQ; footprint Package_SO:SOIC-8_5.23x5.23mm_P1.27mm -> Package_SO:SOIC-8_5.3x5.3mm_P1.27mm; symbol _JLC_Flash_16MB:W25Q16JVSSIQ -> Memory_Flash:W25Q128JVS; LCSC C131025 -> C97521
Other:
- note added: "Flash 128 MBit (16MB)"
- note removed: "Flash 16 MBit (2MB)"
- note removed: "Maybe use 128MBit (16MB) C97521 instead (Basic Part)? 49ct@30pcs vs 19ct@36pcs"
- moved on the sheet: C12, J4, Q1, R3, R6, U2
