File: v3_rp2040/board/lathecontrol_v3.kicad_sch (KiCad schematic)
At the start: 73 parts, among them J1 Conn_01x05_Male, J2 Conn_01x14_Female, J3 Conn_01x05_Male, J4 Conn_01x04_Male, J5 I2C_EXP, J6 SWD, J7 DEBUG, Q1 MMBT3904, Q2 MMBT3904, U1 RP2040, U10 USBLC6-2SC6, U15 LTV-817S-TA1-C, U16 LTV-817S-TA1-C, U17 LTV-817S-TA1-C, U2 LTV-817S-TA1-C, U3 78L05G-AB3-R, U4 LM358DR2G, U5 W25Q128JVSIQ, U6 TYPEC-304-ACP16, U7 TYPEC-304-ACP16, U8 AMS1117-3.3, U9 LM317_TO-252, Y1 12 Mhz

Commit message: schematic work (with Opus 5.5)
Parts:
- removed R4, R5: 5k1, Resistor_SMD:R_0603_1608Metric, symbol Device:R_Small
- removed R7, R8: 27, Resistor_SMD:R_0603_1608Metric, symbol Device:R_Small
- added C21, C22: 220n, Capacitor_SMD:C_0603_1608Metric, symbol Device:C
- added C23: 10n, Capacitor_SMD:C_0603_1608Metric, symbol Device:C
- added C24: 100n, Capacitor_SMD:C_0603_1608Metric, symbol Device:C
- added C25, C26: 47n, Capacitor_SMD:C_0603_1608Metric, symbol Device:C
- added C27: 10u 50V, Capacitor_SMD:C_1206_3216Metric, symbol Device:C
- added C28: 1u, Capacitor_SMD:C_0603_1608Metric, symbol Device:C
- added D5: BAV99, Package_TO_SOT_SMD:SOT-23, symbol Diode:BAV99
- added D6: SS14, Diode_SMD:D_SMA, symbol Device:D_Schottky
- added F1: 50mA, Fuse:Fuse_1206_3216Metric, symbol Device:Polyfuse
- added J8: VFD, TerminalBlock_Phoenix:TerminalBlock_Phoenix_MKDS-1,5-7-5.08_1x07_P5.08mm_Horizontal, symbol Connector:Screw_Terminal_01x07
- added Q3: AO3400A, Package_TO_SOT_SMD:SOT-23, symbol Transistor_FET:AO3400A
- added R20, R25: 330, Resistor_SMD:R_0603_1608Metric, symbol Device:R
- added R21: 4k7, Resistor_SMD:R_0603_1608Metric, symbol Device:R
- added R22, R23: 22k, Resistor_SMD:R_0603_1608Metric, symbol Device:R
- added R24: 220, Resistor_SMD:R_0603_1608Metric, symbol Device:R
- added R26, R28: 1k, Resistor_SMD:R_0603_1608Metric, symbol Device:R
- added R27: 100k, Resistor_SMD:R_0603_1608Metric, symbol Device:R
- added R29: 10k, Resistor_SMD:R_0603_1608Metric, symbol Device:R
- added R52, R9: 27, Resistor_SMD:R_0603_1608Metric, symbol Device:R_Small
- added R53, R54: 5k1, Resistor_SMD:R_0603_1608Metric, symbol Device:R_Small
Connections:
- net +3V3: now also U15.1, U16.1, R29.1, R53.1, R54.1
- net GND: now also U17.3
- net I2C0_SCL: now also R52.2, R54.2
- net I2C0_SDA: now also R53.2, R9.2
- net I2C0_SDA_MCU: now reaches U1.36 (GPIO24)
- net I2C0_SDA_MCU: now also R9.1
- net at U4.1: now also U4.2 (-), R24.1
- net at U4.3 (+): now also C22.1, R23.2
- net at U15.2: now also R20.2
- net COM_ISO: now reaches U15.3
- net COM_ISO: now also U16.3, U3.2 (GND), U4.4 (V-), U4.5 (+), C21.2, C22.2, C23.2, C24.2, C26.2, C27.2, C28.2, D5.1 (K), J8.2 (Pin_2), Q3.2 (S), R27.2
- net at U15.4: now also R21.2, R22.1
- net I2C0_SCL_MCU: now reaches U1.37 (GPIO25)
- net I2C0_SCL_MCU: now also R52.1
- net at U4.6 (-): now also U4.7
- net VFD_PWM: now reaches U1.31 (GPIO20)
- net VFD_PWM: now also R20.1
- net VFD_RUN: now reaches U1.32 (GPIO21)
- net VFD_RUN: now also R25.1
- net VFD_STAT: now reaches U1.34 (GPIO22)
- net VFD_STAT: now also U17.4, R29.2
- net +5V_ISO: now reaches U3.1 (OUT)
- net +5V_ISO: now also C28.1, R26.1, R28.2
- net V15_ISO: now reaches U3.3 (IN)
- net V15_ISO: now also U4.8 (V+), C24.1, C27.1, D6.1 (K)
- net at U17.1: now also R28.1
- net VFD_SP1: now reaches U17.2
- net VFD_SP1: now also J8.5 (Pin_5)
- net at U16.2: now also R25.2
- net at U16.4: now also C25.1, R26.2
- new net: D6.2 (A), F1.2
- new net: C21.1, R22.2, R23.1
- new net: C26.1, D5.2 (A), Q3.1 (G), R27.1
- new net: C25.2, D5.3 (K)
- new net VFD_10V_REF: J8.7 (Pin_7), R21.1
- new net VFD_24V: F1.1, J8.6 (Pin_6)
- new net VFD_VL1: C23.1, J8.1 (Pin_1), R24.2
- new net VFD_X4: J8.3 (Pin_3), Q3.3 (D)
- no-connect marks 27 -> 25
Other:
- note added: "MCU side (GND)"
- note added: "VFD INTERFACE - galvanically isolated (see vfd-interface-plan.md) - Isolation barrier runs through U15/U16/U17: board slot under each opto, no copper in the keep-out, >= 6-8 mm creepage. - COM_ISO is MAINS POTENTIAL. Never tie COM_ISO/V15_ISO/+5V_ISO to GND, PE or enclosure. - GP20 VFD_PWM: ~1 kHz PWM. LED sinks into the pin -> 100 % duty = 0 V on VL1 (invert in FW). Set pad drive strength to 8 m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"
- note added: "VFD side (COM_ISO)"
- moved on the sheet: C10, C11, C12, C14, C15, C16, C9, H1, H2, H3, H4, H5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

Commit message: 7-> 6 terminals for vfd output (drop reverse)
Parts:
- J12: renamed from J8; footprint TerminalBlock_Phoenix:TerminalBlock_Phoenix_MKDS-1,5-7-5.08_1x07_P5.08mm_Horizontal -> TerminalBlock_Phoenix:TerminalBlock_Phoenix_MKDS-1,5-6_1x06_P5.00mm_Horizontal; symbol Connector:Screw_Terminal_01x07 -> Connector:Screw_Terminal_01x06; LCSC (none) -> C192781; MPN (none) -> WJ127-5.0-06P-14-00A
- renumbered C21 to C33, C22 to C34, C23 to C35, C24 to C36, C25 to C37, C26 to C38, C27 to C39, C28 to C40, R20 to R55, R21 to R56, R22 to R57, R23 to R58, R24 to R59, R25 to R60, R26 to R61, R27 to R62, R28 to R63, R29 to R64
Connections:
- net VFD_10V_REF: now also J12.6 (Pin_6); no longer J12.7 (Pin_7)
- net VFD_24V: now also J12.5 (Pin_5); no longer J12.6 (Pin_6)
- net VFD_SP1: now also J12.4 (Pin_4); no longer J12.5 (Pin_5)
- no-connect marks 25 -> 24

Commit message: schematic bla
Parts:
- added JP1: VFDConnect5V, Connector_PinHeader_2.54mm:PinHeader_1x02_P2.54mm_Vertical, symbol Jumper:Jumper_2_Open
- added JP2: VFDConnectGND, Connector_PinHeader_2.54mm:PinHeader_1x02_P2.54mm_Vertical, symbol Jumper:Jumper_2_Open
- C11: renamed from C9; LCSC C13585 -> C15850
- C12: renamed from C33; footprint Capacitor_SMD:C_0603_1608Metric -> Capacitor_SMD:C_0402_1005Metric; LCSC C21120 -> C16772
- C13: renamed from C34; footprint Capacitor_SMD:C_0603_1608Metric -> Capacitor_SMD:C_0402_1005Metric; LCSC C21120 -> C16772
- C14: renamed from C36; footprint Capacitor_SMD:C_0603_1608Metric -> Capacitor_SMD:C_0402_1005Metric; LCSC C14663 -> C307331
- C15: renamed from C35; footprint Capacitor_SMD:C_0603_1608Metric -> Capacitor_SMD:C_0402_1005Metric; LCSC C57112 -> C15195
- C20: renamed from C12; footprint Capacitor_SMD:C_0603_1608Metric -> Capacitor_SMD:C_0402_1005Metric; LCSC C14663 -> C307331
- C23: renamed from C40; footprint Capacitor_SMD:C_0603_1608Metric -> Capacitor_SMD:C_0402_1005Metric; LCSC C15849 -> C52923
- C24: renamed from C17; footprint Capacitor_SMD:C_0603_1608Metric -> Capacitor_SMD:C_0402_1005Metric; LCSC C14663 -> C1525
- C26: renamed from C19; footprint Capacitor_SMD:C_0603_1608Metric -> Capacitor_SMD:C_0402_1005Metric; LCSC C14663 -> C1525
- C27: renamed from C20; footprint Capacitor_SMD:C_0805_2012Metric -> Capacitor_SMD:C_0402_1005Metric; LCSC C13585 -> C15525
- H1, H2, H3, H4, H5: symbol Mechanical:MountingHole_Pad -> Mechanical:MountingHole; now left out of the parts list
- H6: footprint MountingHole:MountingHole_3mm_Pad -> MountingHole:MountingHole_3mm; symbol Mechanical:MountingHole_Pad -> Mechanical:MountingHole; now left out of the parts list
- JP3: renamed from JP1; footprint Resistor_SMD:R_0603_1608Metric -> Resistor_SMD:R_0402_1005Metric; LCSC C21189 -> C17168
- R10: renamed from R53; footprint Resistor_SMD:R_0603_1608Metric -> Resistor_SMD:R_0402_1005Metric; LCSC C23186 -> C25905
- R11: renamed from R54; footprint Resistor_SMD:R_0603_1608Metric -> Resistor_SMD:R_0402_1005Metric; LCSC C23186 -> C25905
- R13: renamed from R60; footprint Resistor_SMD:R_0603_1608Metric -> Resistor_SMD:R_0402_1005Metric; LCSC C23138 -> C25104
- R15: renamed from R62; footprint Resistor_SMD:R_0603_1608Metric -> Resistor_SMD:R_0402_1005Metric; LCSC C25803 -> C25741
- R16: renamed from R64; footprint Resistor_SMD:R_0603_1608Metric -> Resistor_SMD:R_0402_1005Metric; LCSC C25804 -> C25744
- R18: renamed from R63; footprint Resistor_SMD:R_0603_1608Metric -> Resistor_SMD:R_0402_1005Metric; LCSC C21190 -> C11702
- R22: renamed from R13; footprint Resistor_SMD:R_0603_1608Metric -> Resistor_SMD:R_0402_1005Metric; LCSC C23186 -> C25905
- R23: renamed from R14; footprint Resistor_SMD:R_0603_1608Metric -> Resistor_SMD:R_0402_1005Metric; LCSC C23186 -> C25905
- R24: renamed from R15; footprint Resistor_SMD:R_0603_1608Metric -> Resistor_SMD:R_0402_1005Metric; LCSC C23186 -> C25905
- R25: renamed from R16; footprint Resistor_SMD:R_0603_1608Metric -> Resistor_SMD:R_0402_1005Metric; LCSC C23186 -> C25905
- R3: renamed from R56; footprint Resistor_SMD:R_0603_1608Metric -> Resistor_SMD:R_0402_1005Metric; LCSC C23162 -> C25900
- R4: renamed from R57; footprint Resistor_SMD:R_0603_1608Metric -> Resistor_SMD:R_0402_1005Metric; LCSC C31850 -> C25768
- R5: renamed from R58; footprint Resistor_SMD:R_0603_1608Metric -> Resistor_SMD:R_0402_1005Metric; LCSC C31850 -> C25768
- R6: renamed from R59; footprint Resistor_SMD:R_0603_1608Metric -> Resistor_SMD:R_0402_1005Metric; LCSC C22962 -> C25091
- R7: renamed from R55; footprint Resistor_SMD:R_0603_1608Metric -> Resistor_SMD:R_0402_1005Metric; LCSC C23138 -> C25104
- R8: renamed from R61; footprint Resistor_SMD:R_0603_1608Metric -> Resistor_SMD:R_0402_1005Metric; LCSC C21190 -> C11702
- renumbered C11 to C10, C37 to C16, C14 to C17, C15 to C18, C38 to C19, C16 to C21, C39 to C22, C18 to C25, C10 to C9, D5 to D1, D1 to D2, D2 to D3, D3 to D4, D6 to D5, D4 to D6, J5 to J4, J6 to J5, J12 to J6, J4 to J7, J7 to J8, Q3 to Q1, Q1 to Q3, R9 to R12, R52 to R14, R3 to R17, R11 to R19, R12 to R20, R6 to R21, R17 to R26, R18 to R27, R19 to R28, R10 to R9, U15 to U1, U7 to U10, U8 to U11, U9 to U12, U10 to U13, U4 to U2, U1 to U3, U16 to U4, U2 to U5, U17 to U6, U5 to U7, U3 to U8, U6 to U9
Connections:
- net +5V: now also JP1.1 (A)
- net +5V_ISO: now also JP1.2 (B)
- net COM_ISO: now also JP2.1 (A)
- net GND: now also JP2.2 (B); no longer H1.1, H2.1, H3.1, H4.1, H5.1, H6.1
Other:
- note added: "Optional: Take power from VFD"
- note added: "VFD 0...10V Output"
- note added: "VFD Connector"
- note added: "VFD Isolated Side Power"
- note added: "VFD RUN Output with Charge Pump (stop if MCU hangs etc)"
- note added: "VFD Status Read"
- note removed: "MCU side (GND)"
- note removed: "VFD side (COM_ISO)"
- note removed: "https://www.aliexpress.com/item/4001122632293.html"
- moved on the sheet: C11, C12, C13, C14, C15, C16, C19, C20, C22, C23, D1, D5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
