File: v3_rp2040/board/lathecontrol_v3.kicad_pcb (KiCad board)
At the start: 4 copper layers, 99 x 79 mm, 60 parts, among them IC1 LM393, IC2 LM393, IC3 LM393, IC4 LM393, J1 Conn_01x06_Male, J10 USB_A, J11 USB_A, J12 USB_A, J14 Conn_01x04_Male, J4 USB_B_Micro, J5 Conn_01x05_Male, J6 Conn_01x05_Male, J7 Conn_01x14_Female, J9 USB_A, Q2 MMBT3904, U1 STM32F103RBTx, U2 6N137, U4 LM317_TO-252, U5 AMS1117-3.3, Y1 8MHz

Commit message: v3: update PCB from schematic
Pull the resolved footprints, U2/U4/U5 part changes and new datasheet
fields into the board. Project file settings as saved by KiCad.

Co-Authored-By: Claude Opus 5.5 <noreply@anthropic.com>
Parts:
- removed the J1 at (167.0, 140.0)
- removed the J4 at (159.0, 145.5)
- removed the R3 at (199.0, 88.8)
- removed the R6 at (174.4, 123.3)
- removed R9: 13k, Resistor_SMD:R_0603_1608Metric
- added C10: 1u, Capacitor_SMD:C_0402_1005Metric, F.Cu at (123.4, 109.6)
- added C11: 1u, Capacitor_SMD:C_0402_1005Metric, F.Cu at (123.4, 111.6)
- added C14: 22p, Capacitor_SMD:C_0402_1005Metric, F.Cu at (126.3, 103.7)
- added C15: 22p, Capacitor_SMD:C_0402_1005Metric, F.Cu at (126.3, 105.7)
- added C16: 100n, Capacitor_SMD:C_0402_1005Metric, F.Cu at (126.3, 107.6)
- added C21: 220p, Capacitor_SMD:C_0402_1005Metric, F.Cu at (106.3, 123.0)
- added C22: 100n, Capacitor_SMD:C_0402_1005Metric, F.Cu at (106.3, 125.0)
- added C23: 220p, Capacitor_SMD:C_0402_1005Metric, F.Cu at (106.3, 127.0)
- added C24: 220p, Capacitor_SMD:C_0402_1005Metric, F.Cu at (116.4, 123.0)
- added C25: 100n, Capacitor_SMD:C_0402_1005Metric, F.Cu at (116.4, 125.0)
- added C26: 220p, Capacitor_SMD:C_0402_1005Metric, F.Cu at (116.4, 127.0)
- added C27: 220p, Capacitor_SMD:C_0402_1005Metric, F.Cu at (126.5, 123.0)
- added C28: 100n, Capacitor_SMD:C_0402_1005Metric, F.Cu at (126.5, 125.0)
- added C29: 220p, Capacitor_SMD:C_0402_1005Metric, F.Cu at (126.5, 127.0)
- added C30: 220p, Capacitor_SMD:C_0402_1005Metric, F.Cu at (136.5, 123.0)
- added C31: 100n, Capacitor_SMD:C_0402_1005Metric, F.Cu at (136.5, 125.0)
- added C32: 220p, Capacitor_SMD:C_0402_1005Metric, F.Cu at (136.5, 127.0)
- added C8: 100n, Capacitor_SMD:C_0402_1005Metric, F.Cu at (123.4, 107.6)
- added D1: D, Diode_SMD:D_SOD-123F, F.Cu at (121.9, 114.2)
- added J5: I2C_EXP, Connector_PinHeader_2.54mm:PinHeader_1x04_P2.54mm_Vertical, F.Cu at (121.4, 92.8)
- added J6: SWD, Connector_PinHeader_2.54mm:PinHeader_2x03_P2.54mm_Vertical, F.Cu at (108.3, 112.7)
- added J7: DEBUG, Connector_PinHeader_2.54mm:PinHeader_1x04_P2.54mm_Vertical, F.Cu at (126.0, 92.8)
- added Q2: MMBT3904, Package_TO_SOT_SMD:SOT-23, F.Cu at (130.2, 109.6)
- added R13: 5k1, Resistor_SMD:R_0603_1608Metric, F.Cu at (104.0, 104.3)
- added R14: 5k1, Resistor_SMD:R_0603_1608Metric, F.Cu at (104.0, 106.8)
- added R15: 5k1, Resistor_SMD:R_0603_1608Metric, F.Cu at (104.0, 109.3)
- added R16: 5k1, Resistor_SMD:R_0603_1608Metric, F.Cu at (104.0, 111.8)
- added R20: 100k, Resistor_SMD:R_0402_1005Metric, F.Cu at (103.5, 123.1)
- added R21: 33k, Resistor_SMD:R_0402_1005Metric, F.Cu at (103.5, 125.0)
- added R22: 1k, Resistor_SMD:R_0402_1005Metric, F.Cu at (103.5, 127.0)
- added R23: 10k, Resistor_SMD:R_0402_1005Metric, F.Cu at (103.5, 129.0)
- added R24: 100k, Resistor_SMD:R_0402_1005Metric, F.Cu at (103.5, 131.0)
- added R25: 100k, Resistor_SMD:R_0402_1005Metric, F.Cu at (103.5, 133.0)
- added R26: 100k, Resistor_SMD:R_0402_1005Metric, F.Cu at (103.5, 135.0)
- added R27: 1k, Resistor_SMD:R_0402_1005Metric, F.Cu at (103.5, 137.0)
- added R28: 100k, Resistor_SMD:R_0402_1005Metric, F.Cu at (113.5, 123.1)
- added R29: 33k, Resistor_SMD:R_0402_1005Metric, F.Cu at (113.5, 125.0)
- added R30: 1k, Resistor_SMD:R_0402_1005Metric, F.Cu at (113.5, 127.0)
- added R31: 10k, Resistor_SMD:R_0402_1005Metric, F.Cu at (113.5, 129.0)
- added R32: 100k, Resistor_SMD:R_0402_1005Metric, F.Cu at (113.5, 131.0)
- added R33: 100k, Resistor_SMD:R_0402_1005Metric, F.Cu at (113.5, 133.0)
- added R34: 100k, Resistor_SMD:R_0402_1005Metric, F.Cu at (113.5, 135.0)
- added R35: 1k, Resistor_SMD:R_0402_1005Metric, F.Cu at (113.5, 137.0)
- added R36: 100k, Resistor_SMD:R_0402_1005Metric, F.Cu at (123.6, 123.1)
- added R37: 33k, Resistor_SMD:R_0402_1005Metric, F.Cu at (123.6, 125.0)
- added R38: 1k, Resistor_SMD:R_0402_1005Metric, F.Cu at (123.6, 127.0)
- added R39: 10k, Resistor_SMD:R_0402_1005Metric, F.Cu at (123.6, 129.0)
- added R40: 100k, Resistor_SMD:R_0402_1005Metric, F.Cu at (123.6, 131.0)
- added R41: 100k, Resistor_SMD:R_0402_1005Metric, F.Cu at (123.6, 133.0)
- added R42: 100k, Resistor_SMD:R_0402_1005Metric, F.Cu at (123.6, 135.0)
- added R43: 1k, Resistor_SMD:R_0402_1005Metric, F.Cu at (123.6, 137.0)
- added R44: 100k, Resistor_SMD:R_0402_1005Metric, F.Cu at (133.6, 123.1)
- added R45: 33k, Resistor_SMD:R_0402_1005Metric, F.Cu at (133.6, 125.0)
- added R46: 1k, Resistor_SMD:R_0402_1005Metric, F.Cu at (133.6, 127.0)
- added R47: 10k, Resistor_SMD:R_0402_1005Metric, F.Cu at (133.6, 129.0)
- added R48: 100k, Resistor_SMD:R_0402_1005Metric, F.Cu at (133.6, 131.0)
- added R49: 100k, Resistor_SMD:R_0402_1005Metric, F.Cu at (133.6, 133.0)
- added R50: 100k, Resistor_SMD:R_0402_1005Metric, F.Cu at (133.6, 135.0)
- added R51: 1k, Resistor_SMD:R_0402_1005Metric, F.Cu at (133.6, 137.0)
- added TP1: TestPoint, TestPoint:TestPoint_Pad_D1.5mm, F.Cu at (114.9, 112.2)
- added TP2: TestPoint, TestPoint:TestPoint_Pad_D1.5mm, F.Cu at (114.9, 115.7)
- added U10: USBLC6-2SC6, Package_TO_SOT_SMD:SOT-23-6, F.Cu at (130.3, 105.1)
- added U11: USBLC6-2SC6, Package_TO_SOT_SMD:SOT-23-6, F.Cu at (107.5, 130.4)
- added U12: USBLC6-2SC6, Package_TO_SOT_SMD:SOT-23-6, F.Cu at (117.5, 130.4)
- added U13: USBLC6-2SC6, Package_TO_SOT_SMD:SOT-23-6, F.Cu at (127.6, 130.4)
- added U14: USBLC6-2SC6, Package_TO_SOT_SMD:SOT-23-6, F.Cu at (137.7, 130.4)
- added U15: LTV-817S-TA1-C, Package_DIP:SMDIP-4_W9.53mm, F.Cu at (112.6, 93.8)
- added U16: LTV-817S-TA1-C, Package_DIP:SMDIP-4_W9.53mm, F.Cu at (112.6, 100.4)
- added U17: LTV-817S-TA1-C, Package_DIP:SMDIP-4_W9.53mm, F.Cu at (112.6, 107.1)
- added U3: 78L05G-AB3-R, Package_TO_SOT_SMD:SOT-89-3, F.Cu at (128.0, 115.7)
- added U4: LM358DR2G, Package_SO:SOIC-8_3.9x4.9mm_P1.27mm, F.Cu at (139.2, 46.5)
- added U5: W25Q128JVSIQ, Package_SO:SOIC-8_5.3x5.3mm_P1.27mm, F.Cu at (73.2, 116.5)
- added U6: TYPEC-304-ACP16, footprint:USB-C-SMD_TYPE-C-16P-1, F.Cu at (52.8, 85.0)
- added U7: TYPEC-304-ACP16, footprint:USB-C-SMD_TYPE-C-16P-1, F.Cu at (52.8, 94.2)
- C1, C3: value 30p -> 100n; footprint Capacitor_SMD:C_0603_1608Metric -> Capacitor_SMD:C_0402_1005Metric
- C2, C4, C5, C6, C7: footprint Capacitor_SMD:C_0603_1608Metric -> Capacitor_SMD:C_0402_1005Metric
- D2: value RED -> D; footprint LED_SMD:LED_0603_1608Metric -> Diode_SMD:D_SOD-123F
- J10: renamed from J11; footprint Lathecontrol_STM32:USB_A_Upright_C26235 -> footprint:USB_A_Upright_C26235
- J11: renamed from J12; footprint Lathecontrol_STM32:USB_A_Upright_C26235 -> footprint:USB_A_Upright_C26235
- J8: renamed from J9; footprint Lathecontrol_STM32:USB_A_Upright_C26235 -> footprint:USB_A_Upright_C26235
- J9: renamed from J10; footprint Lathecontrol_STM32:USB_A_Upright_C26235 -> footprint:USB_A_Upright_C26235
- JP1: value BOOTSEL -> Auto-Bootsel; footprint Connector_PinHeader_2.54mm:PinHeader_1x02_P2.54mm_Horizontal -> Resistor_SMD:R_0603_1608Metric
- R1: value 10k -> 22; footprint Resistor_SMD:R_0603_1608Metric -> Resistor_SMD:R_0402_1005Metric
- R10: value 3k3 -> 1k; footprint Resistor_SMD:R_0603_1608Metric -> Resistor_SMD:R_0402_1005Metric
- R11: value 13k -> 1k; footprint Resistor_SMD:R_0603_1608Metric -> Resistor_SMD:R_0402_1005Metric
- R12: value 3k3 -> 10k; footprint Resistor_SMD:R_0603_1608Metric -> Resistor_SMD:R_0402_1005Metric
- R2: value 180 -> 22; footprint Resistor_SMD:R_0603_1608Metric -> Resistor_SMD:R_0402_1005Metric
- R4: value 240 -> 5k1
- R5: value 13k -> 5k1
- R7: value 13k -> 27
- R8: value 3k3 -> 27
- U1: value STM32F103RBTx -> RP2040; footprint Package_QFP:LQFP-64_10x10mm_P0.5mm -> footprint:RP2040-QFN-56
- U2: value 6N137 -> LTV-817S-TA1-C; footprint Package_DIP:DIP-8_W7.62mm -> Package_DIP:SMDIP-4_W9.53mm
- Y1: value 8MHz -> 12 Mhz; footprint Crystal:Crystal_SMD_5032-2Pin_5.0x3.2mm -> footprint:OSC-SMD_4P-L3.2-W2.5-BL
- moved U2 136.6 mm to (141.5, 39.8)
- moved C6 117.6 mm to (123.4, 103.7)
- moved R2 112.7 mm to (129.7, 93.5)
- moved Y1 112.5 mm to (61.0, 93.0), turned to 0 degrees
- moved R7 88.3 mm to (104.0, 99.3), turned to 0 degrees
- moved U1 86.3 mm to (100.6, 84.1)
- moved R11 84.9 mm to (129.7, 97.5), turned to 0 degrees
- moved R8 84.0 mm to (104.0, 101.8), turned to 0 degrees
- moved R12 80.7 mm to (129.7, 99.5), turned to 0 degrees
- moved R5 78.8 mm to (104.0, 96.8), turned to 0 degrees
- moved C7 72.6 mm to (123.4, 105.7)
- moved R4 72.0 mm to (104.0, 94.3), turned to 0 degrees
- moved C2 71.9 mm to (120.5, 105.7)
- moved R10 71.9 mm to (129.7, 95.5), turned to 0 degrees
- moved C5 64.1 mm to (120.5, 111.6), turned to 0 degrees
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- renumbered C23 to C12, C20 to C17, C21 to C18, C18 to C19, C19 to C20, C12 to C9, D5 to D3, D6 to D4, J5 to J1, J7 to J2, J6 to J3, J14 to J4, Q2 to Q1, R22 to R17, R20 to R18, R21 to R19, R25 to R3, R26 to R6, U5 to U8, U4 to U9
Connections:
- C1 pad 1: /OSC_IN -> +1V1
- C17 pad 1: +5V -> Net-(D1-K)
- C2 pad 1: +3V3 -> +1V1
- C3 pad 1: /OSC_OUT -> +3V3
- C6 pad 1: Net-(U2-VCC) -> +3V3
- C6 pad 2: unconnected-(C6-Pad2) -> GND
- D2 pad 1: GND -> Net-(D1-K)
- D2 pad 2: Net-(D2-A) -> VBUS
- IC1 pad 2: /Measurestick Input 1/IN_Thres1 -> Net-(IC1A--)
- IC1 pad 3: /Measurestick Input 1/IN_Dat -> /Calipers1/IN_Thres1
- IC1 pad 5: /Measurestick Input 1/IN_Clk -> /Calipers1/IN_Thres1
- IC1 pad 6: /Measurestick Input 1/IN_Thres1 -> Net-(IC1B-_)
- IC2 pad 2: /Measurestick Input 2/IN_Thres1 -> Net-(IC2A--)
- IC2 pad 3: /Measurestick Input 2/IN_Dat -> /Calipers2/IN_Thres1
- IC2 pad 5: /Measurestick Input 2/IN_Clk -> /Calipers2/IN_Thres1
- IC2 pad 6: /Measurestick Input 2/IN_Thres1 -> Net-(IC2B-_)
- IC3 pad 2: /Measurestick Input 3/IN_Thres1 -> Net-(IC3A--)
- IC3 pad 3: /Measurestick Input 3/IN_Dat -> /Calipers3/IN_Thres1
- IC3 pad 5: /Measurestick Input 3/IN_Clk -> /Calipers3/IN_Thres1
- IC3 pad 6: /Measurestick Input 3/IN_Thres1 -> Net-(IC3B-_)
- IC4 pad 2: /Measurestick Input 4/IN_Thres1 -> Net-(IC4A--)
- IC4 pad 3: /Measurestick Input 4/IN_Dat -> /Calipers4/IN_Thres1
- IC4 pad 5: /Measurestick Input 4/IN_Clk -> /Calipers4/IN_Thres1
- IC4 pad 6: /Measurestick Input 4/IN_Thres1 -> Net-(IC4B-_)
- J10 pad 2: /Measurestick Input 3/IN_Clk -> Net-(J10-D-)
- J10 pad 3: /Measurestick Input 3/IN_Dat -> Net-(J10-D+)
- J10 pad 5: GND -> Chassis
- J11 pad 2: /Measurestick Input 4/IN_Clk -> Net-(J11-D-)
- J11 pad 3: /Measurestick Input 4/IN_Dat -> Net-(J11-D+)
- J11 pad 5: GND -> Chassis
- J8 pad 2: /Measurestick Input 1/IN_Clk -> Net-(J8-D-)
- J8 pad 3: /Measurestick Input 1/IN_Dat -> Net-(J8-D+)
- J8 pad 5: GND -> Chassis
- J9 pad 2: /Measurestick Input 2/IN_Clk -> Net-(J9-D-)
- J9 pad 3: /Measurestick Input 2/IN_Dat -> Net-(J9-D+)
- J9 pad 5: GND -> Chassis
- JP1 pad 1: +3V3 -> Net-(JP1-A)
- JP1 pad 2: /BOOT0 -> /BOOTSEL
- Q1 pad 3: Net-(Q2-C) -> Net-(Q1-C)
- R1 pad 1: GND -> /USB_DP2
- R1 pad 2: /BOOT0 -> /USB_DP3
- R10 pad 1: /Measurestick Input 3/IN_Thres1 -> Net-(C15-Pad1)
- R10 pad 2: GND -> /XOUT
- R11 pad 1: +3V3 -> /BOOTSEL
- R11 pad 2: /Measurestick Input 4/IN_Thres1 -> /QSPI_SS
- R12 pad 1: /Measurestick Input 4/IN_Thres1 -> VBUS
- R12 pad 2: GND -> Net-(Q2-B)
- R2 pad 1: Net-(U2-A) -> /USB_DN3
- R2 pad 2: PWM_OUT -> /USB_DN2
- R3 pad 1: Net-(R25-Pad1) -> Net-(R3-Pad1)
- R4 pad 1: /LED_STAT1 -> +3V3
- R4 pad 2: Net-(D2-A) -> /I2C0_SDA
- R5 pad 2: /Measurestick Input 1/IN_Thres1 -> /I2C0_SCL
- R7 pad 1: +3V3 -> Net-(U1-GPIO24)
- R7 pad 2: /Measurestick Input 2/IN_Thres1 -> /I2C0_SDA
- R8 pad 1: /Measurestick Input 2/IN_Thres1 -> Net-(U1-GPIO25)
- R8 pad 2: GND -> /I2C0_SCL
- U1 pad 10: ADC3 -> +3V3
- U1 pad 11: ADC4 -> unconnected-(U1-GPIO8-Pad11)
- U1 pad 12: GND -> unconnected-(U1-GPIO9-Pad12)
- U1 pad 13: +3.3VA -> unconnected-(U1-GPIO10-Pad13)
- U1 pad 14: unconnected-(U1-PA0-Pad14) -> /LED
- U1 pad 15: /LED_STAT1 -> unconnected-(U1-GPIO12-Pad15)
- U1 pad 16: MS1_DAT -> unconnected-(U1-GPIO13-Pad16)
- U1 pad 17: MS1_CLK -> unconnected-(U1-GPIO14-Pad17)
- U1 pad 18: GND -> unconnected-(U1-GPIO15-Pad18)
- U1 pad 19: +3V3 -> GND
- U1 pad 2: ROT1 -> /DBG_TX
- U1 pad 20: MS2_DAT -> /XIN
- U1 pad 21: MS2_CLK -> /XOUT
- U1 pad 22: MS3_DAT -> +3V3
- U1 pad 23: MS3_CLK -> +1V1
- U1 pad 24: unconnected-(U1-PC4-Pad24) -> /SWCLK
- U1 pad 25: unconnected-(U1-PC5-Pad25) -> /SWDIO
- U1 pad 26: MS4_DAT -> /RUN
- U1 pad 27: MS4_CLK -> unconnected-(U1-GPIO16-Pad27)
- U1 pad 29: DISPL_LED -> unconnected-(U1-GPIO18-Pad29)
- U1 pad 3: unconnected-(U1-PC14-Pad3) -> /DBG_RX
- U1 pad 30: DISPL_T_IRQ -> unconnected-(U1-GPIO19-Pad30)
- U1 pad 31: GND -> unconnected-(U1-GPIO20-Pad31)
- U1 pad 32: +3V3 -> unconnected-(U1-GPIO21-Pad32)
- U1 pad 33: unconnected-(U1-PB12-Pad33) -> +3V3
- U1 pad 34: DISPL_SCK -> unconnected-(U1-GPIO22-Pad34)
- U1 pad 35: DISPL_MISO -> unconnected-(U1-GPIO23-Pad35)
- U1 pad 36: DISPL_MOSI -> Net-(U1-GPIO24)
- U1 pad 37: DISPL_CS -> Net-(U1-GPIO25)
- U1 pad 38: DISPL_RST -> unconnected-(U1-GPIO26_ADC0-Pad38)
- U1 pad 39: DISPL_DC -> unconnected-(U1-GPIO27_ADC1-Pad39)
- U1 pad 40: DISPL_T_CS -> unconnected-(U1-GPIO28_ADC2-Pad40)
- U1 pad 41: ENC_BTN -> unconnected-(U1-GPIO29_ADC3-Pad41)
- U1 pad 42: ENC_1 -> +3V3
- U1 pad 43: ENC_2 -> +3V3
- U1 pad 44: USB_D- -> +3V3
- U1 pad 45: USB_D+ -> +1V1
- U1 pad 46: SWDIO -> /USB_DN3
- U1 pad 47: GND -> /USB_DP3
- U1 pad 49: SWCLK -> +3V3
- U1 pad 5: /OSC_IN -> unconnected-(U1-GPIO3-Pad5)
- U1 pad 50: unconnected-(U1-PA15-Pad50) -> +1V1
- U1 pad 51: BTN4 -> /QSPI_SD3
- U1 pad 52: BTN3 -> /QSPI_SCLK
- U1 pad 53: unconnected-(U1-PC12-Pad53) -> /QSPI_SD0
- U1 pad 54: unconnected-(U1-PD2-Pad54) -> /QSPI_SD2
- U1 pad 55: SWD_SWO -> /QSPI_SD1
- U1 pad 56: BTN2 -> /QSPI_SS
- U1 pad 57: BTN1 -> GND
- U1 pad 6: /OSC_OUT -> unconnected-(U1-GPIO4-Pad6)
- U1 pad 7: NRST -> unconnected-(U1-GPIO5-Pad7)
- U1 pad 8: ADC1 -> unconnected-(U1-GPIO6-Pad8)
- U1 pad 9: ADC2 -> unconnected-(U1-GPIO7-Pad9)
- U2 pad 1: unconnected-(U2-NC-Pad1) -> Net-(R3-Pad1)
- U2 pad 2: Net-(U2-A) -> Net-(Q1-C)
- U2 pad 4: (no net) -> ROT1
- U8 pad 3: +5V -> Net-(D1-K)
- Y1 pad 1: /OSC_IN -> /XIN
- Y1 pad 2: /OSC_OUT -> GND
Routing:
- net (no net): track 0.00 -> 786.4 mm, vias 0 -> 14
- net USB_D+: track 92.0 -> 0.00 mm, vias 2 -> 0
- net USB_D-: track 91.3 -> 0.00 mm, vias 2 -> 0
- net SWD_SWO: track 64.3 -> 0.00 mm, vias 2 -> 0
- net SWCLK: track 63.2 -> 0.00 mm, vias 2 -> 0
- net SWDIO: track 58.9 -> 0.00 mm, vias 2 -> 0
- net NRST: track 48.2 -> 0.00 mm
- net ADC2: track 23.7 -> 0.00 mm, vias 1 -> 0
- net ADC1: track 23.4 -> 0.00 mm, vias 1 -> 0
- net ADC3: track 23.0 -> 0.00 mm, vias 1 -> 0
- net ADC4: track 21.3 -> 0.00 mm, vias 1 -> 0
- net /Measurestick Input 3/IN_Dat: track 18.8 -> 0.00 mm
- net /Measurestick Input 1/IN_Dat: track 18.8 -> 0.00 mm
- net /Measurestick Input 2/IN_Dat: track 18.8 -> 0.00 mm
- net /Measurestick Input 4/IN_Dat: track 18.8 -> 0.00 mm
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- removed copper zone on F.Cu, net +3.3VA
